File: NFC_Business_Card.kicad_pcb (KiCad board)
At the start: 2 copper layers, 85.6 x 54 mm, 9 parts, among them U1 ST25DV04KC-IE6T3

Commit message: Added iniital back text
Other:
- board text added: "Scan or Tap"
Changed lines of the file:
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@@
 		)
+	)
+	(gr_text "Mechatronics"
+		(at 62 70 0)
+		(layer "B.SilkS")
+		(effects
+			(font
+				(size 1.2 1.2)
+				(thickness 0.16)
+			)
+			(justify left bottom mirror)
+		)
+	)
+	(gr_text "Cyber Security"
+		(at 62 78 0)
+		(layer "B.SilkS")
+		(effects
+			(font
+				(size 1.2 1.2)
+				(thickness 0.16)
+			)
+			(justify left bottom mirror)
+		)
+	)
+	(gr_text "ryan.yensch.com"
+		(at 62 87 0)
+		(layer "B.SilkS")
+		(effects
+			(font
+				(size 1.2 1.2)
+				(thickness 0.16)
+			)
+			(justify left bottom mirror)
+		)
+	)
+	(gr_text "ryan@yensch.com"
+		(at 62 91 0)
+		(layer "B.SilkS")
+		(effects
+			(font
+				(size 1.2 1.2)
+				(thickness 0.16)
+			)
+			(justify left bottom mirror)
+		)
+	)
+	(gr_text "Software"
+		(at 62 74 0)
+		(layer "B.SilkS")
+		(effects
+			(font
+				(size 1.2 1.2)
+				(thickness 0.16)
+				(bold yes)
+			)
+			(justify left bottom mirror)
+		)
+	)
+	(gr_text "Scan or Tap"
+		(at 115 95 0)
+		(layer "B.SilkS")
+		(effects
+			(font
+				(size 1.3 1.3)
+				(thickness 0.18)
+			)
+			(justify bottom mirror)
+		)
+	)
+	(gr_text "Ryan Yensch"
+		(at 62 63 0)
+		(layer "B.SilkS")
+		(effects
+			(font
+				(size 2.2 2.2)
+				(thickness 0.3)
+			)
+			(justify left bottom mirror)
+		)
+	)
+	(barcode
+		(at 115 76.99 0)
+		(layer "B.SilkS")
+		(size 20 20)
+		(text "https://ryan.yensch.com/nfc")
+		(text_height 1)
+		(type qr)
+		(ecc_level M)
+		(hide yes)
+		(knockout no)
 	)
 	(segment
